File: Untitled/Untitled.kicad_pcb (KiCad board)
At the start: 2 copper layers, 55 x 55 mm, 32 parts, among them J1 Conn_01x02, SW1 MX_SW_HS, SW2 MX_SW_HS, SW4 RST, SW6 MX_SW_HS, SW7 MX_SW_HS, SW8 MX_SW_HS, SW9 MX_SW_HS, U1 nice_nano

Commit message: humidifier
Parts:
- removed J1: Conn_01x02, Connector_JST:JST_PH_S2B-PH-K_1x02_P2.00mm_Horizontal
- moved SW8 14.2 mm to (137.5, 100.0)
- moved D5 14.2 mm to (145.5, 98.9)
- moved D6 13.0 mm to (164.4, 98.8)
- moved SW9 13.0 mm to (156.5, 100.0)
- moved D3 12.9 mm to (145.5, 79.8)
- moved SW6 12.9 mm to (137.5, 81.0)
- moved SW2 11.9 mm to (175.5, 99.9)
- moved D7 11.9 mm to (183.5, 98.7)
- moved D4 11.5 mm to (164.4, 79.9)
- moved SW7 11.5 mm to (156.5, 80.9)
- moved D2 10.2 mm to (183.5, 79.9)
- moved SW1 10.2 mm to (175.5, 80.9)
- moved C1 0.51 mm to (164.8, 56.2)
- moved C7 0.51 mm to (158.8, 56.2)
- moved R5 0.51 mm to (154.5, 56.2)
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Routing:
- net col0: track 46.9 -> 0.00 mm
- net col2: track 40.4 -> 0.00 mm
- net col1: track 35.0 -> 0.00 mm
- net row1: track 70.1 -> 38.5 mm, vias 3 -> 0
- net +3.3V: track 29.5 -> 52.4 mm
- net row0: track 54.5 -> 38.7 mm, vias 4 -> 0
- net GND: track 0.00 -> 14.5 mm, vias 0 -> 10
- net /SCL: track 11.3 -> 13.6 mm
- net Net-(DS1-D/~{C}): track 13.6 -> 12.4 mm
- net /SDA: track 13.7 -> 14.3 mm
- added copper zone on B.Cu, net +3.3V
Other:
- board outline removed

Commit message: idk
Parts:
- moved D3 10.4 mm to (152.7, 72.3)
- moved D4 10.4 mm to (171.6, 72.4)
- moved D6 10.4 mm to (171.6, 91.3)
- moved SW2 10.4 mm to (182.7, 92.5)
- moved SW8 10.4 mm to (144.7, 92.5)
- moved SW9 10.4 mm to (163.7, 92.5)
- moved SW6 10.4 mm to (144.7, 73.5)
- moved SW7 10.4 mm to (163.7, 73.5)
- moved D2 10.4 mm to (190.7, 72.4)
- moved D5 10.4 mm to (152.7, 91.4)
- moved D7 10.4 mm to (190.7, 91.2)
- moved SW1 10.4 mm to (182.7, 73.4)
- moved SW4 2.13 mm to (139.4, 54.4)
- moved U1 2.13 mm to (155.1, 54.2)
- moved C2 2.02 mm to (158.8, 56.2)
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Routing:
- net col0: track 0.00 -> 49.9 mm
- net col2: track 0.00 -> 46.9 mm, vias 0 -> 2
- net col1: track 0.00 -> 40.4 mm, vias 0 -> 2
- net row1: track 38.5 -> 78.1 mm
- net row0: track 38.7 -> 73.4 mm
- net +3.3V: track 52.4 -> 49.0 mm
- net ROT2: track 22.0 -> 25.2 mm
- net ROT1: track 30.5 -> 32.9 mm
- net Net-(DS1-D/~{C}): track 12.4 -> 11.6 mm
- net GND: track 14.5 -> 14.8 mm, vias 10 -> 327
- added copper zone on B.Cu, net GND
- added copper zone on F.Cu, net GND
Other:
- board outline added: 58 x 58 mm
