File: Untitled/Untitled.kicad_sch (KiCad schematic)
At the start: 32 parts, among them J1 Conn_01x02, SW1 MX_SW_HS, SW2 MX_SW_HS, SW4 RST, SW6 MX_SW_HS, SW7 MX_SW_HS, SW8 MX_SW_HS, SW9 MX_SW_HS, U1 nice_nano

Commit message: humidifier
Parts:
- added C11, C12, C13, C14, C9: 1uF, Capacitor_SMD:C_0805_2012Metric_Pad1.18x1.45mm_HandSolder, symbol Device:C
- added D10, D9: LED, symbol Device:LED
- added J3: USB_C_Receptacle_USB2.0_14P, symbol Connector:USB_C_Receptacle_USB2.0_14P
- added R10, R9: 22, Resistor_SMD:R_0805_2012Metric_Pad1.20x1.40mm_HandSolder, symbol Device:R
- added R11, R13: 100, Resistor_SMD:R_0805_2012Metric_Pad1.20x1.40mm_HandSolder, symbol Device:R
- added R12: 10k, Resistor_SMD:R_0805_2012Metric_Pad1.20x1.40mm_HandSolder, symbol Device:R
- added R3, R4: 4.7k, Resistor_SMD:R_0805_2012Metric_Pad1.20x1.40mm_HandSolder, symbol Device:R
- added SW3: RST, Button_Switch_SMD:SW_Tactile_SPST_NO_Straight_CK_PTS636Sx25SMTRLFS, symbol Switch:SW_Push_45deg
- added U2: ATmega32U4-A, Package_QFP:TQFP-44_10x10mm_P0.8mm, symbol MCU_Microchip_ATmega:ATmega32U4-A
- added Y1: 16MHz Crystal, symbol Device:Crystal
Connections:
- net GND: now also C11.2, C12.2, C13.2, C14.2, C9.1, D10.1 (K), D9.1 (K), J3.A1 (GND), J3.A12 (GND), J3.B1 (GND), J3.B12 (GND), J3.S1 (SHIELD), R3.2, R4.2, SW3.2, U2.15 (GND), U2.23 (GND), U2.33 (~{HWB}/PE2), U2.35 (GND), U2.43 (GND), U2.5 (UGND)
- new net: D9.2 (A), R11.2
- new net: J3.A5 (CC1), R3.1
- new net: J3.A6 (D+), J3.B6 (D+), R10.1
- new net: J3.A7 (D-), J3.B7 (D-), R9.1
- new net: J3.B5 (CC2), R4.1
- new net: D10.2 (A), R13.2
- new net: C12.1, U2.42 (AREF)
- new net: C9.2, U2.6 (UCAP)
- new net: R13.1, U2.8 (PB0)
- new net +5V: J3.A4 (VBUS), J3.A9 (VBUS), J3.B4 (VBUS), J3.B9 (VBUS), R11.1, R12.2, U2.14 (VCC), U2.24 (AVCC), U2.34 (VCC), U2.44 (AVCC)
- new net D+: R10.2, U2.4 (D+)
- new net D-: R9.2, U2.3 (D-)
- new net RESET: R12.1, SW3.1, U2.13 (~{RESET})
- new net UVCC: C11.1, U2.2 (UVCC), U2.7 (VBUS)
- new net XTAL1: C13.1, U2.17 (XTAL1), Y1.2
- new net XTAL2: C14.1, U2.16 (XTAL2), Y1.1

Commit message: idk
Parts:
- removed C11, C12, C13, C14, C9: 1uF, Capacitor_SMD:C_0805_2012Metric_Pad1.18x1.45mm_HandSolder, symbol Device:C
- removed D10, D9: LED, symbol Device:LED
- removed J3: USB_C_Receptacle_USB2.0_14P, symbol Connector:USB_C_Receptacle_USB2.0_14P
- removed R10, R9: 22, Resistor_SMD:R_0805_2012Metric_Pad1.20x1.40mm_HandSolder, symbol Device:R
- removed R11, R13: 100, Resistor_SMD:R_0805_2012Metric_Pad1.20x1.40mm_HandSolder, symbol Device:R
- removed R12: 10k, Resistor_SMD:R_0805_2012Metric_Pad1.20x1.40mm_HandSolder, symbol Device:R
- removed R3, R4: 4.7k, Resistor_SMD:R_0805_2012Metric_Pad1.20x1.40mm_HandSolder, symbol Device:R
- removed SW3: RST, Button_Switch_SMD:SW_Tactile_SPST_NO_Straight_CK_PTS636Sx25SMTRLFS, symbol Switch:SW_Push_45deg
- removed U2: ATmega32U4-A, Package_QFP:TQFP-44_10x10mm_P0.8mm, symbol MCU_Microchip_ATmega:ATmega32U4-A
- removed Y1: 16MHz Crystal, symbol Device:Crystal
