File: Untitled/with humiditier.kicad_sch (KiCad schematic)
At the start: 48 parts, among them J3 USB_C_Receptacle_USB2.0_14P, Q1 FMMT491A, Q2 FMMT491A, SW1 MX_SW_HS, SW2 MX_SW_HS, SW3 RST, SW4 RST, SW6 MX_SW_HS, SW7 MX_SW_HS, SW8 MX_SW_HS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

Commit message: idk
Parts:
- removed J3: USB_C_Receptacle_USB2.0_14P, symbol Connector:USB_C_Receptacle_USB2.0_14P
- removed R10, R9: 22, Resistor_SMD:R_0805_2012Metric_Pad1.20x1.40mm_HandSolder, symbol Device:R
- removed SW4: RST, Button_Switch_SMD:SW_Tactile_SPST_NO_Straight_CK_PTS636Sx25SMTRLFS, symbol Switch:SW_Push_45deg
- removed U1: nice_nano, nice-nano-kicad:nice_nano, symbol nice_nano:nice_nano
- added J1: 12402012E212A, 12402012E212A:AMPHENOL_12402012E212A, symbol 12402012E212A:12402012E212A
- added R5: 22, Resistor_SMD:R_0805_2012Metric_Pad1.20x1.40mm_HandSolder, symbol Device:R
- D10, D11, D12, D9: footprint (none) -> LED_SMD:LED_0603_1608Metric_Pad1.05x0.95mm_HandSolder
- LS1, LS2: footprint (none) -> Connector_PinHeader_2.54mm:PinHeader_1x02_P2.54mm_Vertical
- R4: value 4.7k -> 22
Connections:
- net +5V: now also J1.A4_B9 (VBUS)
- net D+: now also J1.A6 (D+_A), J1.B6 (D+_B), R5.2; no longer U2.4 (D+)
- net D-: now also R4.2, J1.A7 (D-_A), J1.B7 (D-_B); no longer U2.3 (D-)
- net GND: now also J1.A1_B12 (GND), J1.A8 (SBU1), J1.B1_A12 (GND__1), J1.B8 (SBU2), J1.SH1 (SHIELD), J1.SH2 (SHIELD__1), J1.SH3 (SHIELD__2), J1.SH4 (SHIELD__3); no longer R4.2
- net P1: now also U2.26 (PD6)
- net P2: now also U2.27 (PD7)
- net ROT1: now also U2.25 (PD4)
- net ROT2: now also U2.22 (PD5)
- net col0: now also U2.29 (PB5)
- net col1: now also U2.12 (PB7)
- net col2: now also U2.30 (PB6)
- net row0: now also U2.20 (PD2)
- net row1: now also U2.21 (PD3)
- net CC1: now reaches R3.1
- net CC1: now also J1.A5 (CC1_A), J1.B5 (CC1_B)
- net D-out: now reaches R4.1
- net D-out: now also U2.3 (D-)
- new net D+out: R5.1, U2.4 (D+)
- no-connect marks 2 -> 14
Other:
- note removed: "nRF52840"
- moved on the sheet: D9, Q1, Q2, R11
