File: Untitled/macro devboard ESP32.kicad_pcb (KiCad board)
At the start: 4 copper layers, 65.6 x 57.1 mm, 48 parts, among them J1 12402012E212A, J2 Conn_01x02_Pin, J3 Conn_02x04_Odd_Even, Q1 BSS84LT1G, SW1 MX_SW_HS, SW3 RST, SW6 MX_SW_HS, SW7 MX_SW_HS, SW8 MX_SW_HS, SW9 MX_SW_HS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

Commit message: used keypad, which doesn't work
Parts:
- removed J2: Conn_01x02_Pin, Connector_JST:JST_XH_B2B-XH-A_1x02_P2.50mm_Vertical
- added C1: 100nF, Capacitor_SMD:C_0603_1608Metric_Pad1.08x0.95mm_HandSolder, F.Cu at (202.2, 44.2)
- added G***: LOGO, LOGO, B.Cu at (197.6, 85.2)
- added J4: Conn_01x02_Pin, Connector_JST:JST_PH_S2B-PH-K_1x02_P2.00mm_Horizontal, B.Cu at (216.1, 86.8)
- added SW2: 1825232-1, 1825232-1:1825232-1_TEC, F.Cu at (209.9, 95.0)
- added TP1: VBAT, TestPoint:TestPoint_Pad_D2.0mm, B.Cu at (215.4, 90.9)
- added TP2: GND, TestPoint:TestPoint_Pad_D2.0mm, B.Cu at (213.2, 49.5)
- added TP3: EN, TestPoint:TestPoint_Pad_D2.0mm, B.Cu at (192.9, 92.7)
- added TP4: VBUS, TestPoint:TestPoint_Pad_D2.0mm, B.Cu at (217.0, 57.7)
- added TP5: VDD, TestPoint:TestPoint_Pad_D2.0mm, B.Cu at (217.0, 61.1)
- added TP6: VIN, TestPoint:TestPoint_Pad_D2.0mm, B.Cu at (200.2, 89.5)
- R14: value 2.7k -> PROG
- SW1, SW6, SW7, SW8, SW9: footprint keyswitches:Kailh_socket_MX -> keyswitches:Kailh_socket_MX_optional
- U4: footprint Package_TO_SOT_SMD:SOT-23-5 -> Package_TO_SOT_SMD:SC-74A-5_1.55x2.9mm_P0.95mm
- moved H1 12.8 mm to (202.6, 94.3)
- moved D5 1.20 mm to (233.6, 85.1), turned to -90 degrees
- moved SW3 1.14 mm to (194.7, 92.8)
- moved C6 1.06 mm to (203.2, 83.5)
- moved R10 1.06 mm to (201.7, 83.5)
- moved D6 1.03 mm to (233.6, 75.0), turned to 90 degrees
- moved D3 0.90 mm to (251.9, 85.2), turned to -90 degrees
- moved SW6 0.64 mm to (245.1, 87.6), turned to 0 degrees
- moved SW8 0.64 mm to (226.0, 87.6), turned to 0 degrees
- moved H2 0.52 mm to (215.9, 43.1)
- moved D2 0.44 mm to (251.9, 57.2), turned to 90 degrees
- moved D4 0.21 mm to (251.9, 75.9), turned to 90 degrees
- moved U4 0.12 mm to (197.0, 85.0)
- turned SW1 to 0 degrees
- turned SW7 to 0 degrees
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Routing:
- net col0: track 51.7 -> 83.5 mm
- net col1: track 56.0 -> 81.7 mm
- net VDD: track 38.6 -> 61.9 mm
- net col2: track 54.5 -> 76.1 mm
- net GND: track 44.9 -> 61.5 mm, vias 203 -> 154
- net Net-(D2-A): track 4.35 -> 20.7 mm
- net Net-(D4-A): track 3.80 -> 20.2 mm
- net Net-(D6-A): track 3.82 -> 18.6 mm
- net ROT2: track 28.3 -> 14.3 mm
- net Net-(D5-A): track 4.54 -> 16.0 mm
- net Net-(D3-A): track 4.50 -> 15.7 mm
- net VBAT_IN: track 0.00 -> 4.35 mm, vias 0 -> 1
- net Net-(D11-K): track 12.8 -> 16.8 mm, vias 0 -> 1
- net EN: track 21.6 -> 24.9 mm, vias 2 -> 3
- net IO20/RXD: track 13.7 -> 10.5 mm
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- added copper zone on F.Cu, net VBAT_IN
Other:
- board text added: "+"
- board text added: "20 RX"
- board text added: "21"
- board text added: "21 TX"
- board text added: "Kevin Ying"
- board text added: "Reset"
- board text added: "TX"
- board text added: "灵 键"
- board text removed: "20/RX"
- board text removed: "21/TX"

Commit message: fixed GPIOs for SPI
Parts:
- removed TP3: EN, TestPoint:TestPoint_Pad_D2.0mm
- removed TP4: VBUS, TestPoint:TestPoint_Pad_D2.0mm
- removed TP5: VDD, TestPoint:TestPoint_Pad_D2.0mm
- added BOOT: RST, Button_Switch_SMD:SW_Tactile_SPST_NO_Straight_CK_PTS636Sx25SMTRLFS, F.Cu at (191.4, 87.8)
- moved TP2 7.50 mm to (216.1, 56.5)
- moved C7 4.73 mm to (195.4, 91.5), turned to 180 degrees
- moved R12 4.30 mm to (194.2, 88.5)
- moved SW3 1.91 mm to (194.9, 94.7)
- moved C5 0.36 mm to (194.2, 84.6)
Connections:
- C7 pad 2: EN -> BOOT
- J3 pad 1: IO20/RXD -> IO3
- J3 pad 2: IO21/TXD -> IO2
- J3 pad 3: IO3 -> IO1
- J3 pad 4: IO2 -> GND
- J3 pad 5: IO1 -> IO6
- J3 pad 6: IO0 -> IO7
- LED0 pad 2: IO0 -> LED1
- R12 pad 2: EN -> BOOT
- SW3 pad 2: EN -> BOOT
- SW7 pad 1: col1 -> BOOT
- SW9 pad 1: col1 -> BOOT
- U1 pad 10: ROT2 -> col2
- U1 pad 11: IO20/RXD -> ROT2
- U1 pad 12: IO21/TXD -> ROT1
- U1 pad 18: IO0 -> LED1
- U1 pad 2: EN -> BOOT
- U1 pad 5: row0 -> IO6
- U1 pad 6: col1 -> IO7
- U1 pad 7: col2 -> row0
- U1 pad 8: ROT1 -> BOOT
Routing:
- net BOOT: track 0.00 -> 93.5 mm, vias 0 -> 3
- net col1: track 81.7 -> 0.00 mm, vias 1 -> 0
- net IO0: track 26.8 -> 0.00 mm, vias 1 -> 0
- net EN: track 24.9 -> 0.00 mm, vias 3 -> 0
- net col2: track 76.1 -> 52.0 mm
- net ROT1: track 42.4 -> 19.2 mm
- net IO7: track 0.00 -> 15.4 mm, vias 0 -> 1
- net IO21/TXD: track 14.4 -> 0.00 mm
- net IO6: track 0.00 -> 14.1 mm, vias 0 -> 1
- net VDD: track 61.9 -> 49.8 mm
- net IO20/RXD: track 10.5 -> 0.00 mm
- net row0: track 83.1 -> 79.4 mm
- net LED1: track 0.00 -> 3.46 mm, vias 0 -> 1
- net GND: track 61.5 -> 63.6 mm, vias 154 -> 151
- net VBUS: track 23.1 -> 21.5 mm, vias 1 -> 0
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Other:
- board text added: "6"
- board text added: "7"
- board text added: "RESET"
- board text removed: "0"
- board text removed: "20 RX"
- board text removed: "21"
- board text removed: "21 TX"
- board text removed: "Reset"
- board text removed: "TX"
